File: pcb/backlight.kicad_pcb (KiCad board)
At the start: 2 copper layers, 100 x 96 mm, 59 parts, among them J3 PJ-002B, J6 USB_C_Receptacle_USB2.0, U1 AL8860WT, U2 IP2721, U3 AL8860WT, U4 AL8860WT

Commit message: fix incorrect part number in BOM
Parts:
- J3: value PJ-002B -> PJ-002AH
Changed lines of the file:
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@@
 			)
 		)
-		(property "Value" "PJ-002B"
+		(property "Value" "PJ-002AH"
 			(at 0 15.5 -90)
 			(layer "F.Fab")
@@
 			)
 		)
-		(property "MPN" "PJ-002B"
+		(property "MPN" "PJ-002AH"
 			(at 0 0 90)
 			(unlocked yes)
@@
 		(fp_arc
 			(start 0.618251 0.501857)
-			(mid 0.523038 0.102216)
+			(mid 0.523039 0.102216)
 			(end 0.620848 -0.296798)
 			(stroke
@@
 		(fp_arc
 			(start -0.581749 0.501857)
-			(mid -0.676962 0.102216)
+			(mid -0.676961 0.102216)
 			(end -0.579152 -0.296798)
 			(stroke
