File: pcb/bsl_driver_v1_a/bsl_drv_v1.kicad_sch (KiCad schematic)
At the start: 45 parts, among them J101 2005WR-2x10P, J102 PJ-320D-4A, Q101 BSS138, SW101 TS-1187A, SW102 TS-1187A, SW103 TS-1187A, U101 W25Q16JVSNIQ, U102 RP2040, Y101 ABM8-272-T3

Commit message: remove csv from gitignore, regenerate BOMs and schematics
Parts:
- C101, C102, C103, C104, C105, C106, C107, C108, C115, C116: Category iND87204 Critical -> (none); JLCPCB Basic Y -> (none); Non-Critical Y -> (none)
- C109, C110, C111, C112, C113, C114, FB101, Q101, R103, R104, R105, R106, R107, R108, R109, SW101, SW102, SW103: JLCPCB Basic Y -> (none)
Connections:
- net TH: no longer C116.1, R109.2, U102.39 (GPIO27_ADC1)
- new net TH+: C116.1, R109.2, U102.39 (GPIO27_ADC1)
