File: pcb/bsl_driver_v1_a/driver_channel.kicad_sch (KiCad schematic)
At the start: 10 parts, among them U301 TPS61169

Commit message: remove csv from gitignore, regenerate BOMs and schematics
Parts:
- C301, C302, C304, D301, R301, R302, R303: JLCPCB Basic Y -> (none)
- C303: Category iND87204 Critical -> (none); JLCPCB Basic Y -> (none); Non-Critical Y -> (none)
Changed lines of the file:
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@@
 			)
 		)
-		(property "Description" "RES THICK FILM 1%"
+		(property "Description" ""
 			(at 123.19 116.84 0)
 			(effects
@@
 		)
 		(property "MPN" "0603WAF510KT5E"
-			(at 123.19 116.84 0)
-			(effects
-				(font
-					(size 1.27 1.27)
-				)
-				(hide yes)
-			)
-		)
-		(property "JLCPCB Basic" "Y"
 			(at 123.19 116.84 0)
 			(effects
@@
 			)
 		)
-		(property "JLCPCB Basic" ""
-			(at 123.19 71.755 0)
-			(effects
-				(font
-					(size 1.27 1.27)
-				)
-				(hide yes)
-			)
-		)
 		(pin "1"
 		)
@@
 			)
 		)
-		(property "JLCPCB Basic" "Y"
-			(at 150.495 98.425 0)
-			(effects
-				(font
-					(size 1.27 1.27)
-				)
-				(hide yes)
-			)
-		)
 		(pin "1"
 		)
@@
 			)
 		)
-		(property "JLCPCB Basic" "Y"
-			(at 89.535 98.425 0)
-			(effects
-				(font
-					(size 1.27 1.27)
-				)
-				(hide yes)
-			)
-		)
 		(pin "1"
 		)
@@
 			)
 		)
-		(property "JLCPCB Basic" "Y"
-			(at 112.395 71.755 0)
-			(effects
-				(font
-					(size 1.27 1.27)
-				)
-				(hide yes)
-			)
-		)
 		(pin "1"
 		)
@@
 			)
 		)
-		(property "Footprint Checked" ""
-			(at 144.78 98.425 0)
-			(effects
-				(font
-					(size 1.27 1.27)
-				)
-				(hide yes)
-			)
-		)
-		(property "Non-Critical" "Y"
-			(at 144.78 98.425 0)
-			(effects
-				(font
-					(size 1.27 1.27)
-				)
-				(hide yes)
-			)
-		)
 		(property "Manufacturer" ""
 			(at 144.78 98.425 0)
@@
 			)
 		)
-		(property "Category" "iND87204 Critical "
-			(at 144.78 98.425 0)
-			(effects
-				(font
-					(size 1.27 1.27)
-				)
-				(hide yes)
-			)
-		)
 		(property "LCSC" "C307331"
-			(at 144.78 98.425 0)
-			(effects
-				(font
-					(size 1.27 1.27)
-				)
-				(hide yes)
-			)
-		)
-		(property "JLCPCB Basic" "Y"
 			(at 144.78 98.425 0)
 			(effects
@@
 			)
 		)
-		(property "JLCPCB Basic" ""
-			(at 113.03 98.425 0)
-			(effects
-				(font
-					(size 1.27 1.27)
-				)
-				(hide yes)
-			)
-		)
 		(pin "1"
 		)
@@
 			)
 		)
-		(property "Description" "RES THICK FILM 1%"
+		(property "Description" ""
 			(at 133.35 116.84 0)
 			(effects
@@
 		)
 		(property "MPN" "0603WAF510KT5E"
-			(at 133.35 116.84 0)
-			(effects
-				(font
-					(size 1.27 1.27)
-				)
-				(hide yes)
-			)
-		)
-		(property "JLCPCB Basic" "Y"
 			(at 133.35 116.84 0)
 			(effects
@@
 			)
 		)
-		(property "Description" "RES THICK FILM 1%"
+		(property "Description" ""
 			(at 102.87 104.775 0)
 			(effects
@@
 		)
 		(property "MPN" "0402WGF1002TCE"
-			(at 102.87 104.775 0)
-			(effects
-				(font
-					(size 1.27 1.27)
-				)
-				(hide yes)
-			)
-		)
-		(property "JLCPCB Basic" "Y"
 			(at 102.87 104.775 0)
 			(effects
@@
 			(at 131.445 93.345 0)
 			(effects
-				(font
-					(size 1.27 1.27)
-				)
-				(hide yes)
-			)
-		)
-		(property "JLCPCB Basic" "Y"
-			(at 131.445 93.345 0)
-			(effects
