File: pcb/bsl_driver_v1_b/driver_channel.kicad_sch (KiCad schematic)
At the start: 11 parts, among them U301 TPS61169

Commit message: remove csv from gitignore, regenerate BOMs and schematics
Parts:
- removed R304: 6.8, Resistor_SMD:R_0402_1005Metric, symbol Device:R_US
- C301, C302, C304: JLCPCB Basic Y -> (none)
- C303: Category iND87204 Critical -> (none); JLCPCB Basic Y -> (none); Non-Critical Y -> (none)
- D301: value DSL14 -> SD103AWS; footprint Diode_SMD:D_SOD-123F -> Diode_SMD:D_SOD-323; JLCPCB Basic Y -> (none); LCSC C22466349 -> C7420360; MPN DSL14 -> SD103AWS
- L301: value 27u -> 82u; LCSC C7588756 -> C7588760; MPN CR6028-270M -> CR6028-820M
- R301: value 20k -> 10k; JLCPCB Basic Y -> (none); LCSC C25765 -> C25744; MPN 0402WGF2002TCE -> 0402WGF1002TCE
- R302, R303: value 6.8 -> 5.1; footprint Resistor_SMD:R_0402_1005Metric -> Resistor_SMD:R_0603_1608Metric; LCSC C227211 -> C25197; MPN AC0402FR-076R8L -> 0603WAF510KT5E
Connections:
- net +5V renamed +3V3
- net +3V3: no longer C301.1, L301.1
- new net VBUS: C301.1, L301.1
Other:
- note added: "Iout = 0.08A"
- note removed: "Iout = 0.09A Rsense power dissipation = 18mW"
- title: scanlight v4 pcb -> big scanlight driver pcb
