File: pcb/sl_v4_a/driver_channel.kicad_sch (KiCad schematic)
At the start: 10 parts, among them U112 TPS61169

Commit message: remove csv from gitignore, regenerate BOMs and schematics
Parts:
- added R304: 6.8, Resistor_SMD:R_0402_1005Metric, symbol Device:R_US
- C301: renamed from C161; JLCPCB Basic Y -> (none)
- C302: renamed from C136; JLCPCB Basic Y -> (none)
- C303: renamed from C172; Category iND87204 Critical -> (none); JLCPCB Basic Y -> (none); Non-Critical Y -> (none)
- C304: renamed from C117; JLCPCB Basic Y -> (none)
- D301: renamed from D110; value SD103AWS -> DSL14; footprint Diode_SMD:D_SOD-323 -> Diode_SMD:D_SOD-123F; JLCPCB Basic Y -> (none); LCSC C7420360 -> C22466349; MPN SD103AWS -> DSL14
- L301: renamed from L108; value 82u -> 27u; LCSC C7588760 -> C7588756; MPN CR6028-820M -> CR6028-270M
- R301: renamed from R137; value 10k -> 20k; JLCPCB Basic Y -> (none); LCSC C25744 -> C25765; MPN 0402WGF1002TCE -> 0402WGF2002TCE
- R302: renamed from R112; value 5.1 -> 6.8; footprint Resistor_SMD:R_0603_1608Metric -> Resistor_SMD:R_0402_1005Metric; JLCPCB Basic Y -> (none); LCSC C25197 -> C227211; MPN 0603WAF510KT5E -> AC0402FR-076R8L
- R303: renamed from R116; value 10 -> 6.8; footprint Resistor_SMD:R_0603_1608Metric -> Resistor_SMD:R_0402_1005Metric; JLCPCB Basic Y -> (none); LCSC C22859 -> C227211; MPN 0603WAF100JT5E -> AC0402FR-076R8L
- renumbered U112 to U301
Connections:
- net VBUS is gone; now on net +5V: C301.1, L301.1
- net GND: now also R304.2
- net OUT-: now also R304.1
- net +3V3 renamed +5V
Other:
- note added: "Iout = 0.09A Rsense power dissipation = 18mW"
- note removed: "Iout = 0.06A"
- company: (none) -> jackw01
- title: (none) -> scanlight v4 pcb
