File: pcb/sl_v4_b/driver_channel.kicad_sch (KiCad schematic)
At the start: 11 parts, among them U301 TPS61169

Commit message: remove csv from gitignore, regenerate BOMs and schematics
Parts:
- C301, C302, C304, D301, R301: JLCPCB Basic Y -> (none)
- C303: Category iND87204 Critical -> (none); JLCPCB Basic Y -> (none); Non-Critical Y -> (none)
Changed lines of the file:
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@@
 			)
 		)
-		(property "Description" "RES THICK FILM 1%"
+		(property "Description" ""
 			(at 123.19 116.84 0)
 			(hide yes)
@@
 		)
 		(property "MPN" "CRCW04026R80FKED"
-			(at 123.19 116.84 0)
-			(hide yes)
-			(show_name no)
-			(do_not_autoplace no)
-			(effects
-				(font
-					(size 1.27 1.27)
-				)
-			)
-		)
-		(property "JLCPCB Basic" ""
 			(at 123.19 116.84 0)
 			(hide yes)
@@
 			)
 		)
-		(property "Description" "RES THICK FILM 1%"
+		(property "Description" ""
 			(at 143.51 116.84 0)
 			(hide yes)
@@
 		)
 		(property "MPN" "CRCW04026R80FKED"
-			(at 143.51 116.84 0)
-			(hide yes)
-			(show_name no)
-			(do_not_autoplace no)
-			(effects
-				(font
-					(size 1.27 1.27)
-				)
-			)
-		)
-		(property "JLCPCB Basic" ""
 			(at 143.51 116.84 0)
 			(hide yes)
@@
 			)
 		)
-		(property "JLCPCB Basic" ""
-			(at 123.19 71.755 0)
-			(hide yes)
-			(show_name no)
-			(do_not_autoplace no)
-			(effects
-				(font
-					(size 1.27 1.27)
-				)
-			)
-		)
 		(pin "1"
 		)
@@
 			)
 		)
-		(property "JLCPCB Basic" "Y"
-			(at 150.495 98.425 0)
-			(hide yes)
-			(show_name no)
-			(do_not_autoplace no)
-			(effects
-				(font
-					(size 1.27 1.27)
-				)
-			)
-		)
 		(pin "1"
 		)
@@
 			)
 		)
-		(property "JLCPCB Basic" "Y"
-			(at 89.535 98.425 0)
-			(hide yes)
-			(show_name no)
-			(do_not_autoplace no)
-			(effects
-				(font
-					(size 1.27 1.27)
-				)
-			)
-		)
 		(pin "1"
 		)
@@
 			)
 		)
-		(property "JLCPCB Basic" "Y"
-			(at 112.395 71.755 0)
-			(hide yes)
-			(show_name no)
-			(do_not_autoplace no)
-			(effects
-				(font
-					(size 1.27 1.27)
-				)
-			)
-		)
 		(pin "1"
 		)
@@
 			)
 		)
-		(property "Footprint Checked" ""
-			(at 144.78 98.425 0)
-			(hide yes)
-			(show_name no)
-			(do_not_autoplace no)
-			(effects
-				(font
-					(size 1.27 1.27)
-				)
-			)
-		)
-		(property "Non-Critical" "Y"
-			(at 144.78 98.425 0)
-			(hide yes)
-			(show_name no)
-			(do_not_autoplace no)
-			(effects
-				(font
-					(size 1.27 1.27)
-				)
-			)
-		)
 		(property "Manufacturer" ""
 			(at 144.78 98.425 0)
@@
 			)
 		)
-		(property "Category" "iND87204 Critical "
-			(at 144.78 98.425 0)
-			(hide yes)
-			(show_name no)
-			(do_not_autoplace no)
-			(effects
-				(font
-					(size 1.27 1.27)
-				)
-			)
-		)
 		(property "LCSC" "C307331"
-			(at 144.78 98.425 0)
-			(hide yes)
-			(show_name no)
-			(do_not_autoplace no)
-			(effects
-				(font
-					(size 1.27 1.27)
-				)
-			)
-		)
-		(property "JLCPCB Basic" "Y"
 			(at 144.78 98.425 0)
 			(hide yes)
@@
 			)
 		)
-		(property "JLCPCB Basic" ""
-			(at 113.03 98.425 0)
-			(hide yes)
-			(show_name no)
-			(do_not_autoplace no)
-			(effects
-				(font
-					(size 1.27 1.27)
-				)
-			)
-		)
 		(pin "1"
 		)
@@
 			)
 		)
-		(property "Description" "RES THICK FILM 1%"
+		(property "Description" ""
 			(at 133.35 116.84 0)
 			(hide yes)
@@
 		)
 		(property "MPN" "CRCW04026R80FKED"
-			(at 133.35 116.84 0)
-			(hide yes)
-			(show_name no)
-			(do_not_autoplace no)
-			(effects
-				(font
-					(size 1.27 1.27)
-				)
-			)
-		)
-		(property "JLCPCB Basic" ""
 			(at 133.35 116.84 0)
 			(hide yes)
@@
 			)
 		)
-		(property "Description" "RES THICK FILM 1%"
+		(property "Description" ""
 			(at 102.87 104.775 0)
 			(hide yes)
@@
 		)
 		(property "MPN" "0402WGF2002TCE"
-			(at 102.87 104.775 0)
-			(hide yes)
-			(show_name no)
-			(do_not_autoplace no)
-			(effects
-				(font
-					(size 1.27 1.27)
-				)
-			)
-		)
-		(property "JLCPCB Basic" "Y"
 			(at 102.87 104.775 0)
 			(hide yes)
@@
 			(at 131.445 93.345 0)
 			(hide yes)
-			(show_name no)
-			(do_not_autoplace no)
-			(effects
-				(font
-					(size 1.27 1.27)
-				)
-			)
-		)
-		(property "JLCPCB Basic" "Y"
-			(at 131.445 93.345 0)
-			(hide yes)
