File: pcb/sl_v4_b/sl_v4.kicad_sch (KiCad schematic)
At the start: 52 parts, among them J101 PJ-320D-4A, SW101 SKRTLAE010, SW102 SKRTLAE010, SW103 SKRTLAE010, U101 W25Q16JVSNIQ, U102 RP2040, U103 TLP172GM, U104 TLP172GM, Y101 ABM8-272-T3

Commit message: remove csv from gitignore, regenerate BOMs and schematics
Parts:
- C101, C102, C103, C104, C105, C106, C107, C108, C115, C116: Category iND87204 Critical -> (none); JLCPCB Basic Y -> (none); Non-Critical Y -> (none)
- C109, C110, C111, C112, C113, C114, FB101, R103, R104, R105, R106, R107, R108, R109, R110, R111: JLCPCB Basic Y -> (none)
