File: pcb/sl_v4_b/usb ports.kicad_sch (KiCad schematic)
At the start: 23 parts, among them J201 TYPE-C-31-M-12, J202 TYPE-C-31-M-12, U201 XC6206P332MR-G

Commit message: remove csv from gitignore, regenerate BOMs and schematics
Parts:
- C201, C203, C204, D201, D202, D203, D204, D205, D206, D207, D208, R203, R204, R205, R206: JLCPCB Basic Y -> (none)
- C202, C205: Category iND87204 Critical -> (none); JLCPCB Basic Y -> (none); Non-Critical Y -> (none)
